File: hexatana.kicad_pcb (KiCad board)
At the start: 2 copper layers, 279.5 x 99.3 mm, 117 parts, among them SW1 SW_Push, SW10 SW_Push, SW11 SW_Push, SW12 SW_Push, SW13 SW_Push, SW14 SW_Push, SW15 SW_Push, SW16 SW_Push, SW17 SW_Push, SW18 SW_Push, SW19 SW_Push, SW2 SW_Push, SW20 SW_Push, SW21 SW_Push, SW22 SW_Push, SW23 SW_Push, SW24 SW_Push, SW25 SW_Push, SW26 SW_Push, SW27 SW_Push, SW28 SW_Push, SW29 SW_Push, SW3 SW_Push, SW30 SW_Push, SW31 SW_Push, SW32 SW_Push, SW33 SW_Push, SW34 SW_Push, SW37 SW_Push, SW38 SW_Push, SW4 SW_Push, SW5 SW_Push, SW6 SW_Push, SW7 SW_Push, SW8 SW_Push, SW9 SW_Push, U2 RP2040-Zero

Commit message: rerouting done
Parts:
- moved D32 37.7 mm to (139.8, 68.3)
- moved D31 36.5 mm to (118.2, 99.3)
- moved D30 21.5 mm to (112.9, 108.6)
- moved D15 21.5 mm to (161.2, 99.3)
- moved D29 18.6 mm to (102.1, 90.0), turned to -150 degrees
- moved D17 10.8 mm to (139.8, 99.3), turned to -90 degrees
- moved D35 10.8 mm to (155.9, 108.6), turned to 30 degrees
- moved D16 10.8 mm to (145.1, 108.6), turned to -30 degrees
- moved D28 10.8 mm to (102.1, 108.6), turned to 150 degrees
Routing:
- net r5: track 99.8 -> 242.3 mm, vias 4 -> 8
- net r6: track 84.8 -> 188.6 mm, vias 3 -> 7
- net Net-(D32-A): track 156.4 -> 208.5 mm
- net Net-(D36-A): track 97.6 -> 55.9 mm
- net r4: track 185.4 -> 152.7 mm, vias 5 -> 6
- net Net-(D31-A): track 156.4 -> 127.6 mm
- net Net-(D11-A): track 159.5 -> 131.3 mm
- net r2: track 140.5 -> 116.9 mm
- net Net-(D14-A): track 119.2 -> 100.0 mm
- net +5V: track 188.5 -> 206.1 mm, vias 71 -> 81
- net Net-(D19-A): track 46.8 -> 64.4 mm
- net Net-(D15-A): track 44.7 -> 62.3 mm
- net Net-(D13-A): track 119.8 -> 102.6 mm
- net Net-(D12-A): track 128.9 -> 112.7 mm
- net Net-(D28-A): track 44.9 -> 29.1 mm
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
Commit message: large diodes
Parts:
- D1, D10, D11, D12, D13, D14, D15, D16, D17, D18, D19, D2, D20, D21, D22, D23, D24, D25, D26, D27, D28, D29, D3, D30, D31, D32, D33, D34, D35, D36, D4, D5, D6, D7, D73, D8, D9: footprint Diode_SMD:D_SOD-323_HandSoldering -> Diode_SMD:D_SOD-123
Routing:
- net GND: track 219.3 -> 207.0 mm
- net r4: track 152.7 -> 156.2 mm
- net Net-(D30-A): track 120.9 -> 117.7 mm
- net r5: track 242.3 -> 240.7 mm
- net Net-(D19-A): track 64.4 -> 63.4 mm
- net Net-(D15-A): track 62.3 -> 63.2 mm
- net Net-(D4-A): track 57.8 -> 58.7 mm
- net Net-(D8-A): track 90.7 -> 91.4 mm
- net r3: track 137.7 -> 137.0 mm
- net r6: track 188.6 -> 188.0 mm
- net Net-(D14-A): track 100.0 -> 100.6 mm
