File: hexatana.kicad_sch (KiCad schematic)
At the start: 73 parts, among them SW1 SW_Push, SW10 SW_Push, SW11 SW_Push, SW12 SW_Push, SW13 SW_Push, SW14 SW_Push, SW15 SW_Push, SW16 SW_Push, SW17 SW_Push, SW18 SW_Push, SW19 SW_Push, SW2 SW_Push, SW20 SW_Push, SW21 SW_Push, SW22 SW_Push, SW23 SW_Push, SW24 SW_Push, SW25 SW_Push, SW26 SW_Push, SW27 SW_Push, SW28 SW_Push, SW29 SW_Push, SW3 SW_Push, SW30 SW_Push, SW31 SW_Push, SW32 SW_Push, SW33 SW_Push, SW34 SW_Push, SW37 SW_Push, SW38 SW_Push, SW4 SW_Push, SW5 SW_Push, SW6 SW_Push, SW7 SW_Push, SW8 SW_Push, SW9 SW_Push, U1 tiny2040

Commit message: before hexed-ground
Parts:
- removed U1: tiny2040, tiny2040:tiny2040, symbol tiny2040:tiny2040
- added C1, C2, C3, C4, C5, C6: C, Capacitor_SMD:C_0603_1608Metric_Pad1.08x0.95mm_HandSolder, symbol Device:C
- added D37, D38, D39, D40, D41, D42, D43, D44, D45, D46, D47, D48, D49, D50, D51, D52, D53, D54, D55, D56, D57, D58, D59, D60, D61, D62, D63, D64, D65, D66, D67, D68, D69, D70, D71, D72: SK6812MINI, PCM_marbastlib-various:LED_6028R, symbol PCM_marbastlib-various:SK6812MINI-E
- added D73: D, Diode_SMD:D_SOD-323_HandSoldering, symbol Device:D
- added JP1: SolderJumper_3_Open, Jumper:SolderJumper-3_P1.3mm_Open_RoundedPad1.0x1.5mm, symbol Jumper:SolderJumper_3_Open
- added U2: RP2040-Zero, RP2040-Zero:RP2040 Zero, symbol RP2040-Zero:RP2040-Zero
Connections:
- net c1: now also U2.11 (GP1)
- net c2: now also U2.12 (GP2)
- net c3: now also U2.13 (GP3); no longer SW18.2, SW23.2, SW28.2
- net c4: now also U2.6 (GP27)
- net c5: now also U2.5 (GP28)
- net c6: now also U2.7 (GP26)
- net r1: now also U2.14 (GP4)
- net r2: now also U2.18 (GP8)
- net r3: now also U2.23 (GP9)
- net r4: now also U2.8 (GP15)
- net r5: now also U2.22 (GP10)
- net r6: now also U2.20 (GP12)
- new net: D38.2 (DOUT), D39.3 (DIN)
- new net: D37.2 (DOUT), D38.3 (DIN)
- new net: D54.2 (DOUT), D55.3 (DIN)
- new net: D53.2 (DOUT), D54.3 (DIN)
- new net: D49.2 (DOUT), D50.3 (DIN)
- new net: D48.2 (DOUT), D49.3 (DIN)
- new net: D59.2 (DOUT), D60.3 (DIN)
- new net: D58.2 (DOUT), D59.3 (DIN)
- new net: D66.2 (DOUT), D67.3 (DIN)
- new net: D65.2 (DOUT), D66.3 (DIN)
- new net: D39.2 (DOUT), D40.3 (DIN)
- new net: D73.1 (K), JP1.3 (B)
- new net: D68.2 (DOUT), D69.3 (DIN)
- new net: D67.2 (DOUT), D68.3 (DIN)
- new net: D47.2 (DOUT), D48.3 (DIN)
- new net: D46.2 (DOUT), D47.3 (DIN)
- new net: D37.1 (VDD), JP1.2 (C)
- new net: D42.2 (DOUT), D43.3 (DIN)
- new net: D41.2 (DOUT), D42.3 (DIN)
- new net: D57.2 (DOUT), D58.3 (DIN)
- new net: D56.2 (DOUT), D57.3 (DIN)
- new net: D64.2 (DOUT), D65.3 (DIN)
- new net: D63.2 (DOUT), D64.3 (DIN)
- new net: D71.2 (DOUT), D72.3 (DIN)
- new net: D52.2 (DOUT), D53.3 (DIN)
- new net: D70.2 (DOUT), D71.3 (DIN)
- new net: D50.2 (DOUT), D51.3 (DIN)
- new net: D51.2 (DOUT), D52.3 (DIN)
- new net: D61.2 (DOUT), D62.3 (DIN)
- new net: D60.2 (DOUT), D61.3 (DIN)
- new net: D69.2 (DOUT), D70.3 (DIN)
- new net: D55.2 (DOUT), D56.3 (DIN)
- new net: D62.2 (DOUT), D63.3 (DIN)
- new net: D40.2 (DOUT), D41.3 (DIN)
- new net: D45.2 (DOUT), D46.3 (DIN)
- new net: D43.2 (DOUT), D44.3 (DIN)
- new net: D44.2 (DOUT), D45.3 (DIN)
- new net +5V: C1.1, C2.1, C3.1, C4.1, C5.1, C6.1, D38.1 (VDD), D39.1 (VDD), D40.1 (VDD), D41.1 (VDD), D42.1 (VDD), D43.1 (VDD), D44.1 (VDD), D45.1 (VDD), D46.1 (VDD), D47.1 (VDD), D48.1 (VDD), D49.1 (VDD), D50.1 (VDD), D51.1 (VDD), D52.1 (VDD), D53.1 (VDD), D54.1 (VDD), D55.1 (VDD), D56.1 (VDD), D57.1 (VDD), D58.1 (VDD), D59.1 (VDD), D60.1 (VDD), D61.1 (VDD), D62.1 (VDD), D63.1 (VDD), D64.1 (VDD), D65.1 (VDD), D66.1 (VDD), D67.1 (VDD), D68.1 (VDD), D69.1 (VDD), D70.1 (VDD), D71.1 (VDD), D72.1 (VDD), D73.2 (A), JP1.1 (A), U2.1 (5V)
- new net GND: C1.2, C2.2, C3.2, C4.2, C5.2, C6.2, D37.4 (VSS), D38.4 (VSS), D39.4 (VSS), D40.4 (VSS), D41.4 (VSS), D42.4 (VSS), D43.4 (VSS), D44.4 (VSS), D45.4 (VSS), D46.4 (VSS), D47.4 (VSS), D48.4 (VSS), D49.4 (VSS), D50.4 (VSS), D51.4 (VSS), D52.4 (VSS), D53.4 (VSS), D54.4 (VSS), D55.4 (VSS), D56.4 (VSS), D57.4 (VSS), D58.4 (VSS), D59.4 (VSS), D60.4 (VSS), D61.4 (VSS), D62.4 (VSS), D63.4 (VSS), D64.4 (VSS), D65.4 (VSS), D66.4 (VSS), D67.4 (VSS), D68.4 (VSS), D69.4 (VSS), D70.4 (VSS), D71.4 (VSS), D72.4 (VSS), U2.2 (GND)
- new net c3p: SW18.2, SW23.2, SW28.2, U2.4 (GP29)
- new net rgb: D37.3 (DIN), U2.10 (GP0)
- no-connect marks 0 -> 8
Other:
- moved on the sheet: D1, D10, D11, D12, D13, D14, D15, D16, D17, D18, D19, D2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

Commit message: converted to gemini and added holes for case
Parts:
- removed D73: D, Diode_SMD:D_SOD-323_HandSoldering, symbol Device:D
- removed JP1: SolderJumper_3_Open, Jumper:SolderJumper-3_P1.3mm_Open_RoundedPad1.0x1.5mm, symbol Jumper:SolderJumper_3_Open
- added H1, H2, H3, H4, H5, H6: MountingHole_Pad, MountingHole:MountingHole_2.2mm_M2_DIN965_Pad, symbol Mechanical:MountingHole_Pad
- U2: footprint RP2040-Zero:RP2040 Zero -> PCM_marbastlib-xp-promicroish:Gemini waveshare
Connections:
- net +5V: now also D37.1 (VDD)
- net GND: now also H1.1, H2.1, H3.1, H4.1, H5.1, H6.1
- net rgb: now also U2.24 (RGB); no longer U2.10 (GP0)
- no-connect marks 8 -> 9
